File: insert pcb/PaxInstrument-T400D-header.brd (EAGLE design)
At the start: 66 x 22.9 mm, 0 parts

Commit message: - Not sure what changed. This is still just playing around.
Other:
- board size 66 x 22.9 mm -> 83.8 x 48.3 mm
Changed lines of the file:
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@@
 <setting verticaltext="up"/>
 </settings>
-<grid distance="0.05" unitdist="inch" unit="mil" style="lines" multiple="1" display="yes" altdistance="5" altunitdist="mil" altunit="mil"/>
+<grid distance="100" unitdist="mil" unit="mil" style="lines" multiple="1" display="yes" altdistance="5" altunitdist="mil" altunit="mil"/>
 <layers>
 <layer number="1" name="Top" color="4" fill="1" visible="yes" active="yes"/>
@@
 <wire x1="17.78" y1="6.35" x2="3.81" y2="6.35" width="0.127" layer="20"/>
 <wire x1="3.81" y1="6.35" x2="0" y2="10.16" width="0.127" layer="20"/>
+<wire x1="69.85" y1="48.26" x2="-3.81" y2="48.26" width="0.254" layer="20"/>
+<wire x1="-8.89" y1="43.18" x2="-8.89" y2="33.02" width="0.254" layer="20"/>
+<wire x1="-3.81" y1="27.94" x2="69.85" y2="27.94" width="0.254" layer="20"/>
+<wire x1="74.93" y1="33.02" x2="74.93" y2="43.18" width="0.254" layer="20"/>
+<wire x1="-3.81" y1="48.26" x2="-8.89" y2="43.18" width="0.254" layer="20" curve="90"/>
+<wire x1="-8.89" y1="33.02" x2="-3.81" y2="27.94" width="0.254" layer="20" curve="90"/>
+<wire x1="69.85" y1="27.94" x2="74.93" y2="33.02" width="0.254" layer="20" curve="90"/>
+<wire x1="74.93" y1="43.18" x2="69.85" y2="48.26" width="0.254" layer="20" curve="90"/>
 </plain>
 <attributes>
